File: electronics/batteryAnalyzer/batteryAnalyzer.kicad_sch (KiCad schematic)
At the start: 7 parts

Commit message: further work on circuit
Parts:
- added D? (x2): SB120, Diode_THT:D_DO-41_SOD81_P10.16mm_Horizontal, symbol Diode:SB120
- added J?: BatteryVoltageMeasurement, symbol Connector:Conn_01x02_Male
- added J?: BatteryConnector, symbol Connector:Conn_01x02_Male
- added J?: ChargeDischargeRelay, symbol Connector:Conn_01x03_Male
- added J?: GndRelay, symbol Connector:Conn_01x02_Male
- added J?: PWM, symbol Connector:Conn_01x02_Male
- added J?: SupplyRelay, symbol Connector:Conn_01x02_Male
- added J?: PowerSupply, symbol Connector:Conn_01x02_Male
- added R?: 0.333, symbol Device:R
- added R? (x2): 68k, symbol Device:R
Connections:
- net GND: now also D?.2 (A), D?.2 (A), J?.1 (Pin_1), J?.1 (Pin_1), J?.1 (Pin_1), R?.2
- net at R?.1: now also J?.2 (Pin_2)
- net at Q?.2 (D): now also J?.2 (Pin_2)
- net at Q?.3 (S): now also R?.1
- new net: J?.1 (Pin_1), J?.1 (Pin_1), J?.2 (Pin_2), R?.1
- new net: D?.1 (K), J?.1 (Pin_1), R?.2
- new net: D?.1 (K), J?.2 (Pin_2), R?.1
- new net: J?.1 (Pin_1), J?.2 (Pin_2), J?.3 (Pin_3), R?.2
- new net: J?.2 (Pin_2), J?.2 (Pin_2)
Other:
- note added: "TODO: - Evtl. an den ADC Leitungen noch Stützkondensatoren hinhängen. - Evlt. an den ADC Leitungen noch Spannungsteiler anbringen. - Reichen 5V Supply Spannung? - Prüfen was passiert, wenn wenn ein Relais nicht öffnet - Statt dem GND Relay eine Diode verwenden? - Wäre gut fürs Entladen um Leistung zu verbraten. - Evtl. auch noch einen Leistungswiderstand?"
- moved on the sheet: C?, Q?, R?
